File: PrechargeRelayDriver.sch.kicad_sch (KiCad schematic)
At the start: 7 parts, among them K4 G2RL-2A, K7 G7L-2A-X-SI_DC12, Q3 DMN61D8LQ

Commit message: schematic: Fix incorrect net on precharge relay
Connections:
- net V-ACC: no longer R26.2
- new net V-TS: R26.2
Changed lines of the file:
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@@
 		)
 	)
-	(global_label "V-ACC"
+	(global_label "V-TS"
 		(shape input)
 		(at 152.4 110.49 270)
@@
 		)
 		(property "Intersheetrefs" "${INTERSHEET_REFS}"
-			(at 152.4 117.7926 90)
+			(at 152.4 116.6498 90)
 			(effects
 				(font
@@
 		(dnp no)
 		(property "Reference" "R26"
-			(at 157.48 106.68 90)
+			(at 156.21 105.41 0)
 			(effects
 				(font
@@
 		)
 		(property "Value" "1k"
-			(at 154.94 106.68 90)
-			(effects
-				(font
+			(at 156.21 107.95 0)
+			(effects
+				(font
