File: AIR_Driver.kicad_sch (KiCad schematic)
At the start: 6 parts, among them J9 MolexMicrofitPlus, Q5 DMN61D8LQ, Q6 DMN61D8LQ

Commit message: schematic: Rename hierarchical sheets
Parts:
- renumbered D19 to D18, J9 to J8, Q5 to Q3, Q6 to Q4, R17 to R15, R18 to R16
Changed lines of the file:
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@@
 		(dnp no)
 		(fields_autoplaced yes)
-		(property "Reference" "#PWR050"
+		(property "Reference" "#PWR045"
 			(at 63.5 72.39 0)
 			(effects
@@
 		(instances
 			(project "Precharge_PCB"
-				(path "/c467677d-b98c-4488-bd11-965ef67263b2/1adc5b19-21a4-403c-9ac5-63a929688c7f"
+				(path "/c467677d-b98c-4488-bd11-965ef67263b2/002009e0-fc6e-484e-9acf-1c1ff1f04f91"
 					(reference "#PWR050")
 					(unit 1)
@@
 		(dnp no)
 		(fields_autoplaced yes)
-		(property "Reference" "#PWR053"
+		(property "Reference" "#PWR048"
 			(at 116.84 60.96 0)
 			(effects
@@
 		)
 		(instances
-			(project ""
-				(path "/c467677d-b98c-4488-bd11-965ef67263b2/1adc5b19-21a4-403c-9ac5-63a929688c7f"
+			(project "Precharge_PCB"
+				(path "/c467677d-b98c-4488-bd11-965ef67263b2/002009e0-fc6e-484e-9acf-1c1ff1f04f91"
 					(reference "#PWR053")
 					(unit 1)
@@
 		(dnp no)
 		(fields_autoplaced yes)
-		(property "Reference" "Q6"
+		(property "Reference" "Q4"
 			(at 105.41 96.5199 0)
 			(effects
@@
 		(instances
 			(project "Precharge_PCB"
-				(path "/c467677d-b98c-4488-bd11-965ef67263b2/1adc5b19-21a4-403c-9ac5-63a929688c7f"
+				(path "/c467677d-b98c-4488-bd11-965ef67263b2/002009e0-fc6e-484e-9acf-1c1ff1f04f91"
 					(reference "Q6")
 					(unit 1)
@@
 		(dnp no)
 		(fields_autoplaced yes)
-		(property "Reference" "R18"
+		(property "Reference" "R16"
 			(at 119.38 60.9599 0)
 			(effects
@@
 		(instances
 			(project "Precharge_PCB"
-				(path "/c467677d-b98c-4488-bd11-965ef67263b2/1adc5b19-21a4-403c-9ac5-63a929688c7f"
+				(path "/c467677d-b98c-4488-bd11-965ef67263b2/002009e0-fc6e-484e-9acf-1c1ff1f04f91"
 					(reference "R18")
 					(unit 1)
@@
 		(dnp no)
 		(fields_autoplaced yes)
-		(property "Reference" "#PWR051"
+		(property "Reference" "#PWR046"
 			(at 63.5 95.25 0)
 			(effects
@@
 		(instances
 			(project "Precharge_PCB"
-				(path "/c467677d-b98c-4488-bd11-965ef67263b2/1adc5b19-21a4-403c-9ac5-63a929688c7f"
+				(path "/c467677d-b98c-4488-bd11-965ef67263b2/002009e0-fc6e-484e-9acf-1c1ff1f04f91"
 					(reference "#PWR051")
 					(unit 1)
@@
 		(on_board yes)
 		(dnp no)
-		(property "Reference" "J9"
+		(property "Reference" "J8"
 			(at 125.73 78.7401 0)
 			(effects
@@
 		(instances
 			(project "Precharge_PCB"
-				(path "/c467677d-b98c-4488-bd11-965ef67263b2/1adc5b19-21a4-403c-9ac5-63a929688c7f"
-					(reference "J9")
+				(path "/c467677d-b98c-4488-bd11-965ef67263b2/002009e0-fc6e-484e-9acf-1c1ff1f04f91"
+					(reference "J7")
 					(unit 1)
 				)
@@
 		(dnp no)
 		(fields_autoplaced yes)
-		(property "Reference" "R17"
+		(property "Reference" "R15"
 			(at 66.04 72.3899 0)
 			(effects
@@
 		)
 		(instances
-			(project ""
-				(path "/c467677d-b98c-4488-bd11-965ef67263b2/1adc5b19-21a4-403c-9ac5-63a929688c7f"
+			(project "Precharge_PCB"
+				(path "/c467677d-b98c-4488-bd11-965ef67263b2/002009e0-fc6e-484e-9acf-1c1ff1f04f91"
 					(reference "R17")
 					(unit 1)
@@
 		(on_board yes)
 		(dnp no)
-		(property "Reference" "D19"
+		(property "Reference" "D18"
 			(at 92.71 78.7399 90)
 			(effects
@@
 		(instances
 			(project "Precharge_PCB"
-				(path "/c467677d-b98c-4488-bd11-965ef67263b2/1adc5b19-21a4-403c-9ac5-63a929688c7f"
-					(reference "D19")
+				(path "/c467677d-b98c-4488-bd11-965ef67263b2/002009e0-fc6e-484e-9acf-1c1ff1f04f91"
+					(reference "D17")
 					(unit 1)
 				)
@@
 		(dnp no)
 		(fields_autoplaced yes)
-		(property "Reference" "#PWR054"
+		(property "Reference" "#PWR049"
 			(at 110.49 76.2 0)
 			(effects
@@
 		(instances
 			(project "Precharge_PCB"
-				(path "/c467677d-b98c-4488-bd11-965ef67263b2/1adc5b19-21a4-403c-9ac5-63a929688c7f"
+				(path "/c467677d-b98c-4488-bd11-965ef67263b2/002009e0-fc6e-484e-9acf-1c1ff1f04f91"
 					(reference "#PWR054")
 					(unit 1)
@@
 		(on_board yes)
 		(dnp no)
-		(property "Reference" "Q5"
+		(property "Reference" "Q3"
 			(at 67.31 82.5499 0)
 			(effects
@@
 		(instances
 			(project "Precharge_PCB"
-				(path "/c467677d-b98c-4488-bd11-965ef67263b2/1adc5b19-21a4-403c-9ac5-63a929688c7f"
+				(path "/c467677d-b98c-4488-bd11-965ef67263b2/002009e0-fc6e-484e-9acf-1c1ff1f04f91"
 					(reference "Q5")
 					(unit 1)
@@
 		(dnp no)
 		(fields_autoplaced yes)
-		(property "Reference" "#PWR052"
+		(property "Reference" "#PWR047"
 			(at 101.6 111.76 0)
 			(effects
@@
 		(instances
 			(project "Precharge_PCB"
-				(path "/c467677d-b98c-4488-bd11-965ef67263b2/1adc5b19-21a4-403c-9ac5-63a929688c7f"
+				(path "/c467677d-b98c-4488-bd11-965ef67263b2/002009e0-fc6e-484e-9acf-1c1ff1f04f91"
 					(reference "#PWR052")
 					(unit 1)
