File: Precharge_Relay.kicad_sch (KiCad schematic)
At the start: 8 parts, among them K3 G9EJH-1-E, Q7 DMN61D8LQ, Q8 DMN61D8LQ

Commit message: *: Remove AIR flyback diodes
Parts:
- D21, D23: Dist (none) -> LCSC; Dist # (none) -> C20754788; Mfr (none) -> JSMSEMI; Mfr # (none) -> 1N4007 M7
Changed lines of the file:
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@@
+			)
+		)
+		(property "Dist" "LCSC"
+			(at 99.06 60.96 90)
+			(effects
+				(font
+					(size 1.27 1.27)
+				)
+				(hide yes)
+			)
+		)
+		(property "Dist #" "C20754788"
+			(at 99.06 60.96 90)
+			(effects
+				(font
+					(size 1.27 1.27)
+				)
+				(hide yes)
+			)
+		)
+		(property "Mfr" "JSMSEMI"
+			(at 99.06 60.96 90)
+			(effects
+				(font
+					(size 1.27 1.27)
+				)
+				(hide yes)
+			)
+		)
+		(property "Mfr #" "1N4007 M7"
+			(at 99.06 60.96 90)
+			(effects
+				(font
+					(size 1.27 1.27)
+				)
+				(hide yes)
 			)
 		)
@@
 			(effects
 				(font
+					(size 1.27 1.27)
+				)
+				(hide yes)
+			)
+		)
+		(property "Dist" "LCSC"
+			(at 120.65 78.74 90)
+			(effects
+				(font
+					(size 1.27 1.27)
+				)
+				(hide yes)
+			)
+		)
+		(property "Dist #" "C20754788"
+			(at 120.65 78.74 90)
+			(effects
+				(font
+					(size 1.27 1.27)
+				)
+				(hide yes)
+			)
+		)
+		(property "Mfr" "JSMSEMI"
+			(at 120.65 78.74 90)
+			(effects
+				(font
+					(size 1.27 1.27)
+				)
+				(hide yes)
+			)
+		)
+		(property "Mfr #" "1N4007 M7"
+			(at 120.65 78.74 90)
+			(effects
+				(font
