File: Precharge_Relay.kicad_sch (KiCad schematic)
At the start: 8 parts, among them K3 G9EJH-1-E, Q7 DMN61D8LQ, Q8 DMN61D8LQ

Commit message: bom: Switch from 1N4007 to BYG20J
Parts:
- D21, D23: value 1N4007 -> BYG20J; Dist # C20754788 -> C241925; Mfr JSMSEMI -> VISHAY; Mfr # 1N4007 M7 -> BYG20J-E3/TR
Changed lines of the file:
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@@
 			)
 		)
-		(property "Value" "1N4007"
+		(property "Value" "BYG20J"
 			(at 96.52 62.2299 90)
 			(effects
@@
 			)
 		)
-		(property "Dist #" "C20754788"
-			(at 99.06 60.96 90)
-			(effects
-				(font
-					(size 1.27 1.27)
-				)
-				(hide yes)
-			)
-		)
-		(property "Mfr" "JSMSEMI"
-			(at 99.06 60.96 90)
-			(effects
-				(font
-					(size 1.27 1.27)
-				)
-				(hide yes)
-			)
-		)
-		(property "Mfr #" "1N4007 M7"
+		(property "Dist #" "C241925"
+			(at 99.06 60.96 90)
+			(effects
+				(font
+					(size 1.27 1.27)
+				)
+				(hide yes)
+			)
+		)
+		(property "Mfr" "VISHAY"
+			(at 99.06 60.96 90)
+			(effects
+				(font
+					(size 1.27 1.27)
+				)
+				(hide yes)
+			)
+		)
+		(property "Mfr #" "BYG20J-E3/TR"
 			(at 99.06 60.96 90)
 			(effects
@@
 			)
 		)
-		(property "Value" "1N4007"
+		(property "Value" "BYG20J"
 			(at 123.19 80.01 90)
 			(effects
@@
 			)
 		)
-		(property "Datasheet" "http://www.vishay.com/docs/88503/1n4001.pdf"
-			(at 120.65 78.74 0)
-			(effects
-				(font
-					(size 1.27 1.27)
-				)
-				(hide yes)
-			)
-		)
-		(property "Description" "1000V 1A General Purpose Rectifier Diode, DO-41"
+		(property "Datasheet" ""
+			(at 120.65 78.74 0)
+			(effects
+				(font
+					(size 1.27 1.27)
+				)
+				(hide yes)
+			)
+		)
+		(property "Description" ""
 			(at 120.65 78.74 0)
 			(effects
@@
 			)
 		)
-		(property "Dist #" "C20754788"
-			(at 120.65 78.74 90)
-			(effects
-				(font
-					(size 1.27 1.27)
-				)
-				(hide yes)
-			)
-		)
-		(property "Mfr" "JSMSEMI"
-			(at 120.65 78.74 90)
-			(effects
-				(font
-					(size 1.27 1.27)
-				)
-				(hide yes)
-			)
-		)
-		(property "Mfr #" "1N4007 M7"
-			(at 120.65 78.74 90)
-			(effects
+		(property "Dist #" "C241925"
+			(at 120.65 78.74 90)
+			(effects
+				(font
+					(size 1.27 1.27)
+				)
+				(hide yes)
+			)
+		)
+		(property "Mfr" "VISHAY"
+			(at 120.65 78.74 90)
+			(effects
+				(font
+					(size 1.27 1.27)
+				)
+				(hide yes)
+			)
+		)
+		(property "Mfr #" "BYG20J-E3/TR"
+			(at 120.65 78.74 90)
+			(effects

Commit message: schematic: Update BOM
Parts:
- D21, D23: DigiKey # (none) -> BYG20J-E3/TR3GICT-ND; Dist LCSC -> (none); Dist # C241925 -> (none); LCSC # (none) -> C241925; Mfr VISHAY -> Vishay; Mouser # (none) -> 625-BYG20J-E3/TR3
- D22: DigiKey # (none) -> BZG05C24-M3-08GICT-ND; Dist DigiKey -> (none); Dist # BZG05C24-M3-08GICT-ND -> (none); LCSC # (none) -> C6136237; Mfr VISHAY -> Vishay; Mouser # (none) -> 78-BZG05C24-M3-08
- K3: DigiKey # (none) -> 39-G9EJH-1-P-EDC12-ND; Dist DigiKey -> (none); Dist # 39-G9EJH-1-P-EDC12-ND -> (none); Mouser # (none) -> 653-G9EJH-1-P-EDC12
- Q7, Q8: DigiKey # (none) -> DMN61D8LQ-7DICT-ND; Dist LCSC -> (none); Dist # C5248874 -> (none); LCSC # (none) -> C5248874; Mouser # (none) -> 621-DMN61D8LQ-7
- R20: Dist LCSC -> (none); Dist # C25804 -> (none); LCSC # (none) -> C25804
- R21: DigiKey # (none) -> 4506-APLR1000J1K00SE-ND; Dist DigiKey -> (none); Dist # 4506-APLR1000J1K00SE-ND -> (none)
Changed lines of the file:
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@@
 			)
 		)
-		(property "Dist" "LCSC"
+		(property "Mfr" "Vishay"
 			(at 99.06 60.96 90)
 			(effects
@@
 			)
 		)
-		(property "Dist #" "C241925"
+		(property "Mfr #" "BYG20J-E3/TR"
 			(at 99.06 60.96 90)
 			(effects
@@
 			)
 		)
-		(property "Mfr" "VISHAY"
+		(property "DigiKey #" "BYG20J-E3/TR3GICT-ND"
 			(at 99.06 60.96 90)
 			(effects
@@
 			)
 		)
-		(property "Mfr #" "BYG20J-E3/TR"
+		(property "LCSC #" "C241925"
+			(at 99.06 60.96 90)
+			(effects
+				(font
+					(size 1.27 1.27)
+				)
+				(hide yes)
+			)
+		)
+		(property "Mouser #" "625-BYG20J-E3/TR3"
 			(at 99.06 60.96 90)
 			(effects
@@
 			)
 		)
-		(property "Dist" "LCSC"
+		(property "Mfr" "Vishay"
 			(at 120.65 78.74 90)
 			(effects
@@
 			)
 		)
-		(property "Dist #" "C241925"
+		(property "Mfr #" "BYG20J-E3/TR"
 			(at 120.65 78.74 90)
 			(effects
@@
 			)
 		)
-		(property "Mfr" "VISHAY"
+		(property "DigiKey #" "BYG20J-E3/TR3GICT-ND"
 			(at 120.65 78.74 90)
 			(effects
@@
 			)
 		)
-		(property "Mfr #" "BYG20J-E3/TR"
+		(property "LCSC #" "C241925"
+			(at 120.65 78.74 90)
+			(effects
+				(font
+					(size 1.27 1.27)
+				)
+				(hide yes)
+			)
+		)
+		(property "Mouser #" "625-BYG20J-E3/TR3"
 			(at 120.65 78.74 90)
 			(effects
@@
 			)
 		)
-		(property "Dist" "DigiKey"
-			(at 120.65 87.63 0)
-			(effects
-				(font
-					(size 1.27 1.27)
-				)
-				(hide yes)
-			)
-		)
-		(property "Dist #" "4506-APLR1000J1K00SE-ND"
-			(at 120.65 87.63 0)
-			(effects
-				(font
-					(size 1.27 1.27)
-				)
-				(hide yes)
-			)
-		)
 		(property "Mfr" "C&B/RESI"
 			(at 120.65 87.63 0)
@@
 		)
 		(property "Mfr #" "APLR1000J1K00SE"
+			(at 120.65 87.63 0)
+			(effects
+				(font
+					(size 1.27 1.27)
+				)
+				(hide yes)
+			)
+		)
+		(property "DigiKey #" "4506-APLR1000J1K00SE-ND"
+			(at 120.65 87.63 0)
+			(effects
+				(font
+					(size 1.27 1.27)
+				)
+				(hide yes)
+			)
+		)
+		(property "LCSC #" ""
+			(at 120.65 87.63 0)
+			(effects
+				(font
+					(size 1.27 1.27)
+				)
+				(hide yes)
+			)
+		)
+		(property "Mouser #" ""
 			(at 120.65 87.63 0)
 			(effects
@@
 			)
 		)
-		(property "Dist" "LCSC"
-			(at 107.95 83.82 0)
-			(effects
-				(font
-					(size 1.27 1.27)
-				)
-				(hide yes)
-			)
-		)
-		(property "Dist #" "C5248874"
-			(at 107.95 83.82 0)
-			(effects
-				(font
-					(size 1.27 1.27)
-				)
-				(hide yes)
-			)
-		)
 		(property "Mfr" "DIODES"
 			(at 107.95 83.82 0)
@@
 		)
 		(property "Mfr #" "DMN61D8LQ-7"
+			(at 107.95 83.82 0)
+			(effects
+				(font
+					(size 1.27 1.27)
+				)
+				(hide yes)
+			)
+		)
+		(property "DigiKey #" "DMN61D8LQ-7DICT-ND"
+			(at 107.95 83.82 0)
+			(effects
+				(font
+					(size 1.27 1.27)
+				)
+				(hide yes)
+			)
+		)
+		(property "LCSC #" "C5248874"
+			(at 107.95 83.82 0)
+			(effects
+				(font
+					(size 1.27 1.27)
+				)
+				(hide yes)
+			)
+		)
+		(property "Mouser #" "621-DMN61D8LQ-7"
 			(at 107.95 83.82 0)
 			(effects
@@
 			)
 		)
-		(property "Dist" "LCSC"
-			(at 66.04 58.42 0)
-			(effects
-				(font
-					(size 1.27 1.27)
-				)
-				(hide yes)
-			)
-		)
-		(property "Dist #" "C25804"
-			(at 66.04 58.42 0)
-			(effects
-				(font
-					(size 1.27 1.27)
-				)
-				(hide yes)
-			)
-		)
 		(property "Mfr" "Uni-Royal"
 			(at 66.04 58.42 0)
@@
 		)
 		(property "Mfr #" "0603WAF1002T5E"
+			(at 66.04 58.42 0)
+			(effects
+				(font
+					(size 1.27 1.27)
+				)
+				(hide yes)
+			)
+		)
+		(property "DigiKey #" ""
+			(at 66.04 58.42 0)
+			(effects
+				(font
+					(size 1.27 1.27)
+				)
+				(hide yes)
+			)
+		)
+		(property "LCSC #" "C25804"
+			(at 66.04 58.42 0)
+			(effects
+				(font
+					(size 1.27 1.27)
+				)
+				(hide yes)
+			)
+		)
+		(property "Mouser #" ""
 			(at 66.04 58.42 0)
 			(effects
@@
 			)
 		)
-		(property "Dist" "LCSC"
-			(at 63.5 68.58 0)
-			(effects
-				(font
-					(size 1.27 1.27)
-				)
-				(hide yes)
-			)
-		)
-		(property "Dist #" "C5248874"
-			(at 63.5 68.58 0)
-			(effects
-				(font
-					(size 1.27 1.27)
-				)
-				(hide yes)
-			)
-		)
 		(property "Mfr" "DIODES"
 			(at 63.5 68.58 0)
@@
 		)
 		(property "Mfr #" "DMN61D8LQ-7"
+			(at 63.5 68.58 0)
+			(effects
+				(font
+					(size 1.27 1.27)
+				)
+				(hide yes)
+			)
+		)
+		(property "DigiKey #" "DMN61D8LQ-7DICT-ND"
+			(at 63.5 68.58 0)
+			(effects
+				(font
+					(size 1.27 1.27)
+				)
+				(hide yes)
+			)
+		)
+		(property "LCSC #" "C5248874"
+			(at 63.5 68.58 0)
+			(effects
+				(font
+					(size 1.27 1.27)
+				)
+				(hide yes)
+			)
+		)
+		(property "Mouser #" "621-DMN61D8LQ-7"
 			(at 63.5 68.58 0)
 			(effects
@@
 			)
 		)
-		(property "Dist" "DigiKey"
-			(at 115.57 64.77 0)
-			(effects
-				(font
-					(size 1.27 1.27)
-				)
-				(hide yes)
-			)
-		)
-		(property "Dist #" "39-G9EJH-1-P-EDC12-ND"
-			(at 115.57 64.77 0)
-			(effects
-				(font
-					(size 1.27 1.27)
-				)
-				(hide yes)
-			)
-		)
 		(property "Mfr" "Omron"
 			(at 115.57 64.77 0)
@@
 		)
 		(property "Mfr #" "G9EJH-1-P-E DC12"
+			(at 115.57 64.77 0)
+			(effects
+				(font
+					(size 1.27 1.27)
+				)
+				(hide yes)
+			)
+		)
+		(property "DigiKey #" "39-G9EJH-1-P-EDC12-ND"
+			(at 115.57 64.77 0)
+			(effects
+				(font
+					(size 1.27 1.27)
+				)
+				(hide yes)
+			)
+		)
+		(property "LCSC #" ""
+			(at 115.57 64.77 0)
+			(effects
+				(font
+					(size 1.27 1.27)
+				)
+				(hide yes)
+			)
+		)
+		(property "Mouser #" "653-G9EJH-1-P-EDC12"
 			(at 115.57 64.77 0)
 			(effects
@@
 			)
 		)
-		(property "Dist" "DigiKey"
-			(at 99.06 69.85 90)
-			(effects
-				(font
-					(size 1.27 1.27)
-				)
-				(hide yes)
-			)
-		)
-		(property "Dist #" "BZG05C24-M3-08GICT-ND"
-			(at 99.06 69.85 90)
-			(effects
-				(font
-					(size 1.27 1.27)
-				)
-				(hide yes)
-			)
-		)
-		(property "Mfr" "VISHAY"
+		(property "Mfr" "Vishay"
 			(at 99.06 69.85 90)
 			(effects
@@
 			(at 99.06 69.85 90)
 			(effects
+				(font
+					(size 1.27 1.27)
+				)
+				(hide yes)
+			)
+		)
+		(property "DigiKey #" "BZG05C24-M3-08GICT-ND"
+			(at 99.06 69.85 90)
+			(effects
+				(font
+					(size 1.27 1.27)
+				)
+				(hide yes)
+			)
+		)
+		(property "LCSC #" "C6136237"
+			(at 99.06 69.85 90)
+			(effects
+				(font
+					(size 1.27 1.27)
+				)
+				(hide yes)
+			)
+		)
+		(property "Mouser #" "78-BZG05C24-M3-08"
+			(at 99.06 69.85 90)
+			(effects
