File: Isolated_Sampler.kicad_sch (KiCad schematic)
At the start: 25 parts, among them U7 AMC1351, U9 TLV6002

Commit message: *: Fix AMC1351 footprint
Parts:
- U7: footprint Package_SO:SOIC-8_3.9x4.9mm_P1.27mm -> Package_SO:SOIC-8_7.5x5.85mm_P1.27mm
Changed lines of the file:
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@@
 			)
 		)
-		(property "Footprint" "Package_SO:SOIC-8_3.9x4.9mm_P1.27mm"
+		(property "Footprint" "Package_SO:SOIC-8_7.5x5.85mm_P1.27mm"
 			(at 77.216 83.566 0)
 			(effects
