File: Isolated_Sampler.kicad_sch (KiCad schematic)
At the start: 25 parts, among them U7 AMC1351, U9 TLV6002

Commit message: schematic: Update BOM
Parts:
- C17, C19, C23: Dist LCSC -> (none); Dist # C5199872 -> (none); LCSC # (none) -> C5199872; Mouser # (none) -> 187-CL10B105KB8NQNC
- C18, C20: DigiKey # (none) -> 1276-1000-1-ND; Dist LCSC -> (none); Dist # C1591 -> (none); LCSC # (none) -> C1591; Mouser # (none) -> 187-CL10B104KB8NNNC
- C21, C22: DigiKey # (none) -> 490-4948-1-ND; LCSC # (none) -> C126579; Mfr (none) -> Murata; Mfr # (none) -> GCM1885C2A331JA16D; Mouser # (none) -> 81-GCM1885C2A331J16D
- C32: DigiKey # (none) -> 490-1451-1-ND; LCSC # (none) -> C77026; Mfr (none) -> Murata; Mfr # (none) -> GRM1885C1H102JA01D; Mouser # (none) -> 81-GRM39C102J50
- R38, R39: Dist LCSC -> (none); Dist # C21190 -> (none); LCSC # (none) -> C21190
- TP10, TP8: DigiKey # (none) -> 36-5000-ND; LCSC # (none) -> C5199900; Mfr (none) -> Keystone Electronics; Mfr # (none) -> 5000; Mouser # (none) -> 534-5000
- U7: DigiKey # (none) -> 296-AMC1351QDWVRQ1CT-ND; Dist Mouser -> (none); Dist # 595-AMC1351QDWVRQ1 -> (none); LCSC # (none) -> C5214207; Mouser # (none) -> 595-AMC1351QDWVRQ1
- U9: DigiKey # (none) -> 296-TLV6002QDRQ1CT-ND; Dist Mouser -> (none); Dist # 595-TLV6002QDRQ1 -> (none); LCSC # (none) -> C1850245; Mouser # (none) -> 595-TLV6002QDRQ1
